File: PCB/Macropad.kicad_sch (KiCad schematic)
At the start: 9 parts, among them SW1 SW_Push, SW2 SW_Push, SW3 SW_Push, SW4 SW_Push, U1 XIAO-RP2040-DIP

Commit message: Added OLED
Parts:
- added U2: ~, OLED:SSD1306-0.91-OLED-4pin-128x32, symbol OPL:OLED_DISPLAY
Connections:
- net +5V: now also U2.2 (VCC)
- net GND: now also U2.1 (GND)
- net at U1.1 (GPIO26/ADC0/A0): now also D1.3 (DIN)
- net SDA: now reaches U1.5 (GPIO6/SDA)
- net SDA: now also U2.4 (SDA); no longer D1.3 (DIN)
- net SCL: now reaches U1.6 (GPIO7/SCL)
- net SCL: now also U2.3 (SCL)
